Commit message: PROJECT SETTING

File: src/project01/urdf/robot.xacro (robot description, xacro)
@@ -49,16 +49,16 @@
     </joint>
     <joint name="joint_chassis_front_left_wheel" type="continuous">
-        <origin rpy="0 0 0" xyz="0.5 0.65 0" />
+        <origin rpy="0 0 0" xyz="0.5 0.83 0" />
         <child link="link_front_left_wheel" />
         <parent link="link_chassis" />
-        <axis rpy="0 0 0" xyz="0 1 0" />
+        <axis rpy="0 0 0" xyz="0 0 1" />
         <limit effort="10000" velocity="1000" />
         <joint_properties damping="1.0" friction="1.0" />
     </joint>
     <joint name="joint_chassis_front_right_wheel" type="continuous">
-        <origin rpy="0 0 0" xyz="0.5 -0.65 0" />
+        <origin rpy="0 0 0" xyz="0.5 -0.83 0" />
         <child link="link_front_right_wheel" />
         <parent link="link_chassis" />
-        <axis rpy="0 0 0" xyz="0 1 0" />
+        <axis rpy="0 0 0" xyz="0 0 1" />
         <limit effort="10000" velocity="1000" />
         <joint_properties damping="1.0" friction="1.0" />
@@ -154,18 +154,18 @@
             <!-- Wheel -->
         <collision>
-            <origin rpy="${PI/2} 0 0" xyz="0 0.18 0" />
-            <geometry>
-                <mesh filename="package://robot_description/meshes/wheel.stl" />
-            </geometry>
-        </collision>
-        <visual>
-            <origin rpy="${PI/2} 0 0" xyz="0 0.18 0" />
-            <geometry>
-                <mesh filename="package://robot_description/meshes/wheel.stl" />
-            </geometry>
-            <material name="black"/>
-        </visual>
-        <visual>
-            <origin rpy="0 0 0" xyz="0 0.18 0" />
+            <origin rpy="${PI/2} 0 0" xyz="0 0 0" />
+            <geometry>
+                <mesh filename="package://robot_description/meshes/wheel.stl" />
+            </geometry>
+        </collision>
+        <visual>
+            <origin rpy="${PI/2} 0 0" xyz="0 0 0" />
+            <geometry>
+                <mesh filename="package://robot_description/meshes/wheel.stl" />
+            </geometry>
+            <material name="black"/>
+        </visual>
+        <visual>
+            <origin rpy="0 0 0" xyz="0 0 0" />
             <geometry>
                 <box size="0.1 0.1 0.7" />
@@ -175,15 +175,9 @@
             <!-- Shaft -->
         <collision>
-            <origin rpy="${PI/2} 0 0" xyz="0 0.06 0" />
-            <geometry>
-                <cylinder length="0.12" radius="0.08"/>
-            </geometry>
-        </collision>
-        <visual>
-            <origin rpy="${PI/2} 0 0" xyz="0 0.06 0" />
-            <geometry>
-                <cylinder length="0.12" radius="0.08"/>
-            </geometry>
-        </visual>
+            <origin rpy="${PI/2} 0 0" xyz="0 -0.12 0" />
+            <geometry>
+                <cylinder length="0.12" radius="0.08"/>
+            </geometry>
+        </collision>
     </link>
     <link name="link_front_right_wheel">
@@ -195,35 +189,22 @@
             <!-- Wheel -->
         <collision>
-            <origin rpy="${PI/2} 0 0" xyz="0 -0.18 0" />
-            <geometry>
-                <mesh filename="package://robot_description/meshes/wheel.stl" />
-            </geometry>
-        </collision>
-        <visual>
-            <origin rpy="${PI/2} 0 0" xyz="0 -0.18 0" />
-            <geometry>
-                <mesh filename="package://robot_description/meshes/wheel.stl" />
-            </geometry>
-            <material name="black"/>
-        </visual>
-        <visual>
-            <origin rpy="0 0 0" xyz="0 -0.18 0" />
-            <geometry>
-                <box size="0.1 0.1 0.7" />
-            </geometry>
-            <material name="grey"/>
-        </visual>
-            <!-- Shaft -->
-        <collision>
-            <origin rpy="${PI/2} 0 0" xyz="0 -0.06 0" />
-            <geometry>
-                <cylinder length="0.12" radius="0.08"/>
-            </geometry>
-        </collision>
-        <visual>
-            <origin rpy="${PI/2} 0 0" xyz="0 -0.06 0" />
-            <geometry>
-                <cylinder length="0.12" radius="0.08"/>
-            </geometry>
+            <origin rpy="${PI/2} 0 0" xyz="0 0 0" />
+            <geometry>
+                <mesh filename="package://robot_description/meshes/wheel.stl" />
+            </geometry>
+        </collision>
+        <visual>
+            <origin rpy="${PI/2} 0 0" xyz="0 0 0" />
+            <geometry>
+                <mesh filename="package://robot_description/meshes/wheel.stl" />
+            </geometry>
+            <material name="black"/>
+        </visual>
+        <visual>
+            <origin rpy="0 0 0" xyz="0 0 0" />
+            <geometry>
+                <box size="0.1 0.1 0.7" />
+            </geometry>
+            <material name="grey"/>
         </visual>
     </link>
@@ -262,3 +243,23 @@
         </collision>
     </link>
+    <transmission name="tran_front_left_wheel">
+        <type>transmission_interface/SimpleTransmission</type>
+        <joint name="joint_chassis_front_left_wheel">
+            <hardwareInterface>hardware_interface/EffortJointInterface</hardwareInterface>
+        </joint>
+        <actuator name="motor_front_left_wheel">
+            <hardwareInterface>hardware_interface/EffortJointInterface</hardwareInterface>
+            <mechanicalReduction>1</mechanicalReduction>
+        </actuator>
+    </transmission>
+    <transmission name="tran_front_right_wheel">
+        <type>transmission_interface/SimpleTransmission</type>
+        <joint name="joint_chassis_front_right_wheel">
+            <hardwareInterface>hardware_interface/EffortJointInterface</hardwareInterface>
+        </joint>
+        <actuator name="motor_front_right_wheel">
+            <hardwareInterface>hardware_interface/EffortJointInterface</hardwareInterface>
+            <mechanicalReduction>1</mechanicalReduction>
+        </actuator>
+    </transmission>
 </robot>
