Commit message: Done

File: src/robot_description/urdf/robot.xacro (robot description, xacro)
@@ -2,14 +2,15 @@
 <robot name="robot" xmlns:xacro="http://www.ros.org/wiki/xacro">
     <xacro:include filename="$(find robot_description)/urdf/robot.gazebo" />
+    <xacro:property name="PI" value="3.1415926535"/>
     <material name="blue">
-        <color rgba="0 0 0.8 0.5"/>
+        <color rgba="0 0 0.8 1"/>
     </material>
     <material name="black">
-        <color rgba="0 0 0 0.8"/>
+        <color rgba="0 0 0 1"/>
     </material>
     <material name="grey">
-        <color rgba="0.5 0.5 0.5 0.5"/>
+        <color rgba="0.5 0.5 0.5 1"/>
     </material>
-    <!-- Link - chassis -->
+    <!-- Link - chassis (Model Body) -->
     <link name="link_chassis">
         <inertial>
@@ -20,151 +21,182 @@
         <collision>
             <geometry>
-                <box size="2 1.3 0.4" />
-            </geometry>
-        </collision>
-        <visual>
-            <geometry>
-                <box size="2 1.3 0.4" />
-            </geometry>
-            <material name="blue"/>
-        </visual>
-    </link>
-            <!-- Joint - chassis / left wheel -->
-        <joint name="joint_chassis_left_wheel" type="continuous">
-            <origin rpy="0 0 0" xyz="-0.5 0.65 0" />
-            <child link="link_left_wheel" />
-            <parent link="link_chassis" />
-            <axis rpy="0 0 0" xyz="0 1 0" />
-            <limit effort="10000" velocity="1000" />
-            <joint_properties damping="1.0" friction="1.0" />
-        </joint>
-        <joint name="joint_chassis_right_wheel" type="continuous">
-            <origin rpy="0 0 0" xyz="-0.5 -0.65 0" />
-            <child link="link_right_wheel" />
-            <parent link="link_chassis" />
-            <axis rpy="0 0 0" xyz="0 1 0" />
-            <limit effort="10000" velocity="1000" />
-            <joint_properties damping="1.0" friction="1.0" />
-        </joint>
-        <!-- Link - left wheel -->
-        <link name="link_left_wheel">
-            <inertial>
-                <mass value="1" />
-                <origin xyz="0 0 0" rpy="0 0 0" />
-                <inertia ixx="0.002526666666667" ixy="0" ixz="0" iyy="0.002526666666667" iyz="0" izz="0.005"/>
-            </inertial>
-                <!-- Wheel -->
-            <collision>
-                <origin rpy="1.5708 0 0" xyz="0 0.18 0" />
-                <geometry>
-                    <cylinder length="0.12" radius="0.4"/>
-                </geometry>
-            </collision>
-            <visual>
-                <origin rpy="1.5708 0 0" xyz="0 0.18 0" />
-                <geometry>
-                    <cylinder length="0.12" radius="0.4"/>
-                </geometry>
-                <material name="black"/>
-            </visual>
-            <visual>
-                <origin rpy="0 0 0" xyz="0 0.18 0" />
-                <geometry>
-                    <box size="0.1 1 0.5" />
-                </geometry>
+                <mesh filename="package://robot_description/meshes/chassis.stl" />
+            </geometry>
+            <material name="grey">
+                <color rgba="0.5 0.5 0.5 0.5"/>
+            </material>
+        </collision>
+        <visual>
+            <geometry>
+                <mesh filename="package://robot_description/meshes/chassis.stl" />
+            </geometry>
+        </visual>
+    </link>
+    <!-- Joint - chassis / Wheel -->
+    <joint name="joint_chassis_left_wheel" type="continuous">
+        <origin rpy="0 0 0" xyz="-0.5 0.65 0" />
+        <child link="link_left_wheel" />
+        <parent link="link_chassis" />
+        <axis rpy="0 0 0" xyz="0 1 0" />
+        <limit effort="10000" velocity="1000" />
+        <joint_properties damping="1.0" friction="1.0" />
+    </joint>
+    <joint name="joint_chassis_right_wheel" type="continuous">
+        <origin rpy="0 0 0" xyz="-0.5 -0.65 0" />
+        <child link="link_right_wheel" />
+        <parent link="link_chassis" />
+        <axis rpy="0 0 0" xyz="0 1 0" />
+        <limit effort="10000" velocity="1000" />
+        <joint_properties damping="1.0" friction="1.0" />
+    </joint>
+    <!-- Link - left wheel -->
+    <link name="link_left_wheel">
+        <inertial>
+            <mass value="1" />
+            <origin xyz="0 0 0" rpy="0 0 0" />
+            <inertia ixx="0.002526666666667" ixy="0" ixz="0" iyy="0.002526666666667" iyz="0" izz="0.005"/>
+        </inertial>
+            <!-- Wheel -->
+        <collision>
+            <origin rpy="${PI/2} 0 0" xyz="0 0.18 0" />
+            <geometry>
+                <mesh filename="package://robot_description/meshes/wheel.stl" />
+            </geometry>
+        </collision>
+        <visual>
+            <origin rpy="${PI/2} 0 0" xyz="0 0.18 0" />
+            <geometry>
+                <mesh filename="package://robot_description/meshes/wheel.stl" />
+            </geometry>
+        </visual>
+        <visual>
+            <origin rpy="0 0 0" xyz="0 0.18 0" />
+            <geometry>
+                <box size="0.1 0.1 0.7" />
+            </geometry>
+            <material name="grey"/>
+        </visual>
+            <!-- Shaft -->
+        <collision>
+            <origin rpy="${PI/2} 0 0" xyz="0 0.06 0" />
+            <geometry>
+                <cylinder length="0.12" radius="0.08"/>
+            </geometry>
+        </collision>
+        <visual>
+            <origin rpy="${PI/2} 0 0" xyz="0 0.06 0" />
+            <geometry>
+                <cylinder length="0.12" radius="0.08"/>
+            </geometry>
+        </visual>
+    </link>
+    <link name="link_right_wheel">
+        <inertial>
+            <mass value="1" />
+            <origin xyz="0 0 0" rpy="0 0 0" />
+            <inertia ixx="0.002526666666667" ixy="0" ixz="0" iyy="0.002526666666667" iyz="0" izz="0.005"/>
+        </inertial>
+            <!-- Wheel -->
+        <collision>
+            <origin rpy="${PI/2} 0 0" xyz="0 -0.18 0" />
+            <geometry>
+                <mesh filename="package://robot_description/meshes/wheel.stl" />
+            </geometry>
+        </collision>
+        <visual>
+            <origin rpy="${PI/2} 0 0" xyz="0 -0.18 0" />
+            <geometry>
+                <mesh filename="package://robot_description/meshes/wheel.stl" />
+            </geometry>
+        </visual>
+        <visual>
+            <origin rpy="0 0 0" xyz="0 -0.18 0" />
+            <geometry>
+                <box size="0.1 0.1 0.7" />
                 <material name="grey"/>
-            </visual>
-                <!-- Shaft -->
-            <collision>
-                <origin rpy="1.5708 0 0" xyz="0 0.06 0" />
-                <geometry>
-                    <cylinder length="0.12" radius="0.08"/>
-                </geometry>
-            </collision>
-            <visual>
-                <origin rpy="1.5708 0 0" xyz="0 0.06 0" />
-                <geometry>
-                    <cylinder length="0.12" radius="0.08"/>
-                </geometry>
-                <material name="black"/>
-            </visual>
-        </link>
-        <link name="link_right_wheel">
-            <inertial>
-                <mass value="1" />
-                <origin xyz="0 0 0" rpy="0 0 0" />
-                <inertia ixx="0.002526666666667" ixy="0" ixz="0" iyy="0.002526666666667" iyz="0" izz="0.005"/>
-            </inertial>
-                <!-- Wheel -->
-            <collision>
-                <origin rpy="1.5708 0 0" xyz="0 -0.18 0" />
-                <geometry>
-                    <cylinder length="0.12" radius="0.4"/>
-                </geometry>
-            </collision>
-            <visual>
-                <origin rpy="1.5708 0 0" xyz="0 -0.18 0" />
-                <geometry>
-                    <cylinder length="0.12" radius="0.4"/>
-                </geometry>
-                <material name="black"/>
-            </visual>
-            <visual>
-                <origin rpy="0 0 0" xyz="0 -0.18 0" />
-                <geometry>
-                    <box size="0.1 1 0.5" />
-                </geometry>
+            </geometry>
+        </visual>
+            <!-- Shaft -->
+        <collision>
+            <origin rpy="${PI/2} 0 0" xyz="0 -0.06 0" />
+            <geometry>
+                <cylinder length="0.12" radius="0.08"/>
+            </geometry>
+        </collision>
+        <visual>
+            <origin rpy="${PI/2} 0 0" xyz="0 -0.06 0" />
+            <geometry>
+                <cylinder length="0.12" radius="0.08"/>
+            </geometry>
+        </visual>
+    </link>
+    <!-- Spherical Wheel -->
+    <joint name="joint_spherical_wheel" type="fixed">
+        <origin rpy="0 0 0" xyz="0.7 0 -0.15" />
+        <child link="link_spherical_wheel" />
+        <parent link="link_chassis" />
+        <axis rpy="0 0 0" xyz="0 1 0" />
+        <limit effort="10000" velocity="1000" />
+        <joint_properties damping="1.0" friction="1.0" />
+    </joint>
+    <link name="link_spherical_wheel">
+        <inertial>
+            <mass value="1" />
+            <origin xyz="0 0 0" rpy="0 0 0" />
+            <inertia ixx="0.002526666666667" ixy="0" ixz="0" iyy="0.002526666666667" iyz="0" izz="0.005"/>
+        </inertial>
+            <!-- Wheel -->
+        <collision>
+            <origin rpy="0 0 0" xyz="0 0 -0.125" />
+            <geometry>
+                <sphere radius="0.125"/>
+            </geometry>
+        </collision>
+        <visual>
+            <origin rpy="0 0 0" xyz="0 0 -0.125" />
+            <geometry>
+                <sphere radius="0.125"/>
+            </geometry>
+        </visual>
+        <visual>
+            <origin rpy="0 0 0" xyz="0 0 -0.05" />
+            <geometry>
+                <sphere radius="0.15"/>
+            </geometry>
                 <material name="grey"/>
-            </visual>
-                <!-- Shaft -->
-            <collision>
-                <origin rpy="1.5708 0 0" xyz="0 -0.06 0" />
-                <geometry>
-                    <cylinder length="0.12" radius="0.08"/>
-                </geometry>
-            </collision>
-            <visual>
-                <origin rpy="1.5708 0 0" xyz="0 -0.06 0" />
-                <geometry>
-                    <cylinder length="0.12" radius="0.08"/>
-                </geometry>
-                <material name="black"/>
-            </visual>
-        </link>
-                <!-- Gazebo tags - Laser scan -->
-        <gazebo reference="joint_laser_scan_chassis">
-            <preserveFixedJoint>true</preserveFixedJoint>
-        </gazebo>
-        <gazebo reference="link_laser_scan">
-            <material>Gazebo/DarkGrey</material>
-        </gazebo>
-        <!-- Laser scan -->
-        <joint name="joint_laser_scan_chassis" type="fixed">
-            <origin rpy="0 0 0" xyz="0.8 0 0.3" />
-            <child link="link_laser_scan" />
-            <parent link="link_chassis" />
-            <joint_properties damping="1.0" friction="1.0" />
-        </joint>
-        <link name="link_laser_scan">
-            <inertial>
-                <origin xyz="0 0 0" rpy="0 0 0" />
-                <mass value="0.5" />
-                <inertia ixx="0.000252666666667" ixy="0" ixz="0" iyy="0.000252666666667" iyz="0" izz="0.0005"/>
-            </inertial>
-            <visual>
-                <origin xyz="0 0 0" rpy="0 0 0" />
-                <geometry>
-                    <cylinder radius="0.15" length="0.20"/>
-                </geometry>
-                <material name="Red">
-                    <color rgba="0.7 0.1 0.1 1" />
-                </material>
-            </visual>
-            <collision>
-                <origin xyz="0 0 0" rpy="0 0 0"/>
-                <geometry>
-                    <cylinder radius="0.15" length="0.20"/>
-                </geometry>
-            </collision>
-        </link>
+        </visual>
+    </link>
+    <!-- Gazebo tags - Laser scan -->
+    <gazebo reference="joint_laser_scan_chassis">
+        <preserveFixedJoint>true</preserveFixedJoint>
+    </gazebo>
+    <gazebo reference="link_laser_scan">
+        <material>Gazebo/DarkGrey</material>
+    </gazebo>
+    <!-- Laser scan -->
+    <joint name="joint_laser_scan_chassis" type="fixed">
+        <origin rpy="0 0 0" xyz="0.8 0 0.3" />
+        <child link="link_laser_scan" />
+        <parent link="link_chassis" />
+        <joint_properties damping="1.0" friction="1.0" />
+    </joint>
+    <link name="link_laser_scan">
+        <inertial>
+            <origin xyz="0 0 0" rpy="0 0 0" />
+            <mass value="0.5" />
+            <inertia ixx="0.000252666666667" ixy="0" ixz="0" iyy="0.000252666666667" iyz="0" izz="0.0005"/>
+        </inertial>
+        <visual>
+            <origin xyz="0 0 0" rpy="0 0 0" />
+            <geometry>
+                <cylinder radius="0.15" length="0.20"/>
+            </geometry>
+        </visual>
+        <collision>
+            <origin xyz="0 0 0" rpy="0 0 0"/>
+            <geometry>
+                <cylinder radius="0.15" length="0.20"/>
+            </geometry>
+        </collision>
+    </link>
 </robot>

Commit message: JOINT TAIL XACRO

File: src/robot_description/urdf/robot.xacro (robot description, xacro)
@@ -200,3 +200,33 @@
         </collision>
     </link>
+        <!-- Robot tail -->
+    <joint name="joint_tail" type="continuous">
+        <origin rpy="0 0 0" xyz="-1 0 0" />
+        <child link="link_tail" />
+        <axis rpy="0 0 0" xyz="0 1 0" />
+        <parent link="link_chassis" />
+        <joint_properties damping="1.0" friction="1.0" />
+    </joint>
+    <link name="link_tail">
+        <inertial>
+            <origin xyz="0 0 0" rpy="0 0 0" />
+            <mass value="0.5" />
+            <inertia ixx="0.000252666666667" ixy="0" ixz="0" iyy="0.000252666666667" iyz="0" izz="0.0005"/>
+        </inertial>
+        <visual>
+            <origin xyz="-0.2 0 0" rpy="0 ${pi/2} 0" />
+            <geometry>
+                <cylinder radius="0.05" length="0.40"/>
+            </geometry>
+            <material name="Red">
+                <color rgba="0.7 0.1 0.1 1" />
+            </material>
+        </visual>
+        <collision>
+            <origin xyz="-0.2 0 0" rpy="0 ${pi/2} 0"/>
+            <geometry>
+                <cylinder radius="0.05" length="0.40"/>
+            </geometry>
+        </collision>
+    </link>
 </robot>

Commit message: TRANSMISSION TAIL

File: src/robot_description/urdf/robot.xacro (robot description, xacro)
@@ -4,5 +4,5 @@
     <xacro:property name="PI" value="3.1415926535"/>
     <material name="blue">
-        <color rgba="0 0 0.8 1"/>
+        <color rgba="0 0 0.8 0.8"/>
     </material>
     <material name="black">
@@ -23,7 +23,4 @@
                 <mesh filename="package://robot_description/meshes/chassis.stl" />
             </geometry>
-            <material name="grey">
-                <color rgba="0.5 0.5 0.5 0.5"/>
-            </material>
         </collision>
         <visual>
@@ -31,4 +28,5 @@
                 <mesh filename="package://robot_description/meshes/chassis.stl" />
             </geometry>
+            <material name="blue"/>
         </visual>
     </link>
@@ -69,4 +67,5 @@
                 <mesh filename="package://robot_description/meshes/wheel.stl" />
             </geometry>
+            <material name="black"/>
         </visual>
         <visual>
@@ -109,4 +108,5 @@
                 <mesh filename="package://robot_description/meshes/wheel.stl" />
             </geometry>
+            <material name="black"/>
         </visual>
         <visual>
@@ -114,6 +114,6 @@
             <geometry>
                 <box size="0.1 0.1 0.7" />
-                <material name="grey"/>
-            </geometry>
+            </geometry>
+            <material name="grey"/>
         </visual>
             <!-- Shaft -->
@@ -158,4 +158,5 @@
                 <sphere radius="0.125"/>
             </geometry>
+            <material name="grey"/>
         </visual>
         <visual>
@@ -164,5 +165,5 @@
                 <sphere radius="0.15"/>
             </geometry>
-                <material name="grey"/>
+                <material name="black"/>
         </visual>
     </link>
@@ -192,4 +193,5 @@
                 <cylinder radius="0.15" length="0.20"/>
             </geometry>
+            <material name="black"/>
         </visual>
         <collision>
@@ -230,3 +232,13 @@
         </collision>
     </link>
+    <transmission name="tran_tail">
+        <type>transmission_interface/SimpleTransmission</type>
+        <joint name="joint_tail">
+            <hardwareInterface>hardware_interface/EffortJointInterface</hardwareInterface>
+        </joint>
+        <actuator name="motor_joint_tail">
+            <hardwareInterface>hardware_interface/EffortJointInterface</hardwareInterface>
+            <mechanicalReduction>1</mechanicalReduction>
+        </actuator>
+    </transmission>
 </robot>

Commit message: Project01 세팅 완료

File: src/robot_description/urdf/robot.xacro (robot description, xacro)
@@ -242,3 +242,23 @@
         </actuator>
     </transmission>
+    <transmission name="tran_wheel1">
+        <type>transmission_interface/SimpleTransmission</type>
+        <joint name="joint_chassis_left_wheel">
+            <hardwareInterface>hardware_interface/EffortJointInterface</hardwareInterface>
+        </joint>
+        <actuator name="actuator_wheel1">
+            <hardwareInterface>hardware_interface/EffortJointInterface</hardwareInterface>
+            <mechanicalReduction>1</mechanicalReduction>
+        </actuator>
+    </transmission>
+    <transmission name="tran_wheel2">
+        <type>transmission_interface/SimpleTransmission</type>
+        <joint name="joint_chassis_right_wheel">
+            <hardwareInterface>hardware_interface/EffortJointInterface</hardwareInterface>
+        </joint>
+        <actuator name="actuator_wheel2">
+            <hardwareInterface>hardware_interface/EffortJointInterface</hardwareInterface>
+            <mechanicalReduction>1</mechanicalReduction>
+        </actuator>
+    </transmission>
 </robot>
